File: Headphone DAC AMP/Headphone DAC AMP.kicad_pcb (KiCad board)
At the start: 2 copper layers, 170 parts, among them J1 2137160001, J2 M50-3551042, J4 PINHD_1x2_Male, J5 PINHD_2x3_Male, U1 ES9039Q2M, U11 ADP5071AREZ-R7, U12 TPS74501PDRVR, U14 ADP7185ACPZN-R7, U2 XU316-1024-QF60B-C24, U4 OPA1612AxD, U5 OPA1612AxD, U6 MCP1727-1802xSN, U7 MCP1727-3302xSN, U9 TPS717XX, Y1 Crystal_GND24, Y2 LMK6CE049152CDLFR, Y3 ASDLJ-E-45.1584MHz

Commit message: Fixed all the work i put in
Parts:
- removed C25, C28, C31: 400p, Capacitor_SMD:C_0805_2012Metric_Pad1.18x1.45mm_HandSolder
- removed C26, C29, C32: 110p, Capacitor_SMD:C_0805_2012Metric_Pad1.18x1.45mm_HandSolder
- removed C27, C30: 1p, Capacitor_SMD:C_0805_2012Metric_Pad1.18x1.45mm_HandSolder
- removed R10, R21, R6: 4.7k, Resistor_SMD:R_0805_2012Metric_Pad1.20x1.40mm_HandSolder
- removed R18, R22, R23, R9: 1k, Resistor_SMD:R_0805_2012Metric_Pad1.20x1.40mm_HandSolder
- removed R19, R7: 4.8k, Resistor_SMD:R_0805_2012Metric_Pad1.20x1.40mm_HandSolder
- removed R20, R5, R8: 4.7meg, Resistor_SMD:R_0805_2012Metric_Pad1.20x1.40mm_HandSolder
- added C103: 1u, Capacitor_SMD:C_0402_1005Metric_Pad0.74x0.62mm_HandSolder, F.Cu at (233.5, 73.1)
- added FB1: 220R, Capacitor_SMD:C_0805_2012Metric_Pad1.18x1.45mm_HandSolder, F.Cu at (234.3, 68.1)
- added FB2: 600R @ 100MHz, Capacitor_SMD:C_0603_1608Metric_Pad1.08x0.95mm_HandSolder, F.Cu at (234.0, 70.9)
- C5: value 400p -> 2200p
- C6, C8: value 1p -> 2200p
- C7: value 110p -> 2200p
- R1, R4: value 4.8k -> 800
- R2: value 4.7meg -> 800
- R3: value 4.7k -> 800
- R41: footprint Inductor_SMD:L_0805_2012Metric -> Resistor_SMD:R_0805_2012Metric_Pad1.20x1.40mm_HandSolder
- moved C8 21.0 mm to (251.0, 110.0), turned to 90 degrees
- moved C7 18.7 mm to (237.5, 108.5), turned to 90 degrees
- moved R3 18.5 mm to (239.5, 108.5), turned to 90 degrees
- moved R4 16.6 mm to (249.0, 110.0)
- moved C6 12.4 mm to (250.8, 89.8), turned to 90 degrees
- moved R2 11.0 mm to (248.8, 89.8), turned to 90 degrees
- moved R1 6.49 mm to (239.2, 88.3), turned to 90 degrees
- moved C5 4.47 mm to (237.2, 88.3), turned to 90 degrees
- moved C85 1.32 mm to (247.8, 85.8)
- moved C86 1.32 mm to (240.2, 94.2)
- moved C89 1.32 mm to (245.8, 85.8)
- moved C90 1.32 mm to (241.2, 94.2)
- moved C93 1.32 mm to (246.8, 85.8)
- moved C94 1.32 mm to (242.2, 94.2)
- moved U4 1.22 mm to (244.1, 89.8)
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Connections:
- net /Power Managment/+5V5 renamed /Audio Rails/+5V5
- net /Power Managment/-5V5 renamed /Audio Rails/-5V5
- net /Power Managment/-5VFB renamed /Audio Rails/-5VFB
- net /Power Managment/5VFB renamed /Audio Rails/5VFB
- net /Power Managment/VREF renamed /Audio Rails/VREF
- net /Power Managment/VREG renamed /Audio Rails/VREG
- net Net-(Y2-OUT) renamed /Clocking/MCLK
- C10 pad 1: /USB Audio Input/0V9BP -> 0V9
- C100 pad 1: /USB Audio Input/1V1BP -> +3.3V
- C101 pad 1: /USB Audio Input/1V1BP -> +3.3V
- C102 pad 1: /USB Audio Input/1V1BP -> +3.3V
- C11 pad 1: /USB Audio Input/0V9BP -> 0V9
- C12 pad 1: /USB Audio Input/0V9BP -> 0V9
- C13 pad 1: /USB Audio Input/0V9BP -> 0V9
- C14 pad 1: /USB Audio Input/0V9BP -> 0V9
- C15 pad 1: /USB Audio Input/0V9BP -> 0V9
- C16 pad 1: /USB Audio Input/0V9BP -> 0V9
- C22 pad 1: /Power Managment/+5V_FLT -> /Audio Rails/+5V_FLT
- C42 pad 1: /Power Managment/-5V_FLT -> /Headphone Amp Stage/L+FLT
- C46 pad 1: /Low Noise Rails/Vin -> /Audio Rails/5Vin
- C47 pad 1: /Low Noise Rails/Vin -> /Audio Rails/5Vin
- C5 pad 1: Net-(C5-Pad1) -> /DAC/DAC2b
- C5 pad 2: Net-(U4A-+) -> /Headphone Amp Stage/OUTA
- C50 pad 1: /Power Managment/+5V_FLT -> /Audio Rails/+5V_FLT
- C51 pad 1: /Power Managment/+5V_FLT -> /Audio Rails/+5V_FLT
- C55 pad 1: /Power Managment/-5V_FLT -> /Headphone Amp Stage/L+FLT
- C6 pad 1: Net-(U4A--) -> /DAC/DAC2
- C6 pad 2: GND -> /Headphone Amp Stage/OUTB
- C61 pad 1: /Low Noise Rails/Vin -> /Audio Rails/5Vin
- C68 pad 1: /Headphone Amp Stage/L-FLT -> /Audio Rails/+5V_FLT
- C69 pad 1: /Headphone Amp Stage/L-FLT -> /Audio Rails/+5V_FLT
- C7 pad 1: Net-(C7-Pad1) -> /DAC/DAC1b
- C7 pad 2: GND -> /Headphone Amp Stage/OUTC
- C70 pad 1: /Headphone Amp Stage/L-FLT -> /Audio Rails/+5V_FLT
- C71 pad 1: /Headphone Amp Stage/L-FLT -> /Audio Rails/+5V_FLT
- C72 pad 1: /Headphone Amp Stage/L-FLT -> /Audio Rails/+5V_FLT
- C78 pad 1: /Headphone Amp Stage/L-FLT -> /Audio Rails/+5V_FLT
- C79 pad 1: /Headphone Amp Stage/L-FLT -> /Audio Rails/+5V_FLT
- C8 pad 1: Net-(U4B--) -> /DAC/DAC1
- C8 pad 2: GND -> /Headphone Amp Stage/OUTD
- C80 pad 1: /Headphone Amp Stage/L-FLT -> /Audio Rails/+5V_FLT
- C81 pad 1: /Headphone Amp Stage/L-FLT -> /Audio Rails/+5V_FLT
- C82 pad 1: /Headphone Amp Stage/L-FLT -> /Audio Rails/+5V_FLT
- C84 pad 1: /Headphone Amp Stage/L-FLT -> /Audio Rails/+5V_FLT
- C86 pad 1: /Headphone Amp Stage/L-FLT -> /Audio Rails/+5V_FLT
- C88 pad 1: /Headphone Amp Stage/L-FLT -> /Audio Rails/+5V_FLT
- C9 pad 1: /USB Audio Input/0V9BP -> 0V9
- C90 pad 1: /Headphone Amp Stage/L-FLT -> /Audio Rails/+5V_FLT
- C92 pad 1: /Headphone Amp Stage/L-FLT -> /Audio Rails/+5V_FLT
- C94 pad 1: /Headphone Amp Stage/L-FLT -> /Audio Rails/+5V_FLT
- C96 pad 1: /USB Audio Input/3V3BP -> +1V8
- C97 pad 1: /USB Audio Input/3V3BP -> +1V8
- C98 pad 1: /USB Audio Input/3V3BP -> +1V8
- C99 pad 1: /USB Audio Input/3V3BP -> +1V8
- J4 pad 2: /Low Noise Rails/Vin -> /Audio Rails/5Vin
- R1 pad 2: Net-(C5-Pad1) -> /Headphone Amp Stage/OUTA
- R2 pad 1: Net-(C5-Pad1) -> /DAC/DAC2
- R2 pad 2: Net-(U4A--) -> /Headphone Amp Stage/OUTB
- R3 pad 1: Net-(U4A-+) -> /DAC/DAC1b
- R3 pad 2: Net-(C7-Pad1) -> /Headphone Amp Stage/OUTC
- R33 pad 1: /Power Managment/-5V_FLT -> /Headphone Amp Stage/L+FLT
- R37 pad 1: /Power Managment/+5V_FLT -> /Audio Rails/+5V_FLT
- R39 pad 1: /Power Managment/+5V_FLT -> /Audio Rails/+5V_FLT
- R4 pad 1: /DAC/DAC2 -> /DAC/DAC1
- R4 pad 2: Net-(C25-Pad1) -> /Headphone Amp Stage/OUTD
- U11 pad 11: 5Vin -> /Audio Rails/5Vin
- U11 pad 17: 5Vin -> /Audio Rails/5Vin
- U11 pad 18: 5Vin -> /Audio Rails/5Vin
- U11 pad 19: 5Vin -> /Audio Rails/5Vin
- U11 pad 9: 5Vin -> /Audio Rails/5Vin
- U12 pad 1: /Power Managment/+5V_FLT -> /Audio Rails/+5V_FLT
- U14 pad 1: /Power Managment/-5V_FLT -> /Headphone Amp Stage/L+FLT
- U14 pad 2: /Power Managment/-5V_FLT -> /Headphone Amp Stage/L+FLT
- U2 pad 12: /USB Audio Input/0V9BP -> 0V9
- U2 pad 17: unconnected-(U2-VDDIOB18-Pad17) -> +3.3V
- U2 pad 19: /USB Audio Input/0V9BP -> 0V9
- U2 pad 21: /USB Audio Input/RST_N -> /Debug/XMOS_NRST
- U2 pad 22: unconnected-(U2-PLL_AVDD-Pad22) -> /USB Audio Input/PLL_AVDD
- U2 pad 26: unconnected-(U2-VDDIOB18-Pad26) -> +3.3V
- U2 pad 27: /USB Audio Input/0V9BP -> 0V9
- U2 pad 30: /USB Audio Input/3V3BP -> +1V8
- U2 pad 31: +1V8 -> +3.3V
- U2 pad 34: /USB Audio Input/0V9BP -> 0V9
- U2 pad 38: /USB Audio Input/3V3BP -> +1V8
- U2 pad 4: /USB Audio Input/0V9BP -> 0V9
- U2 pad 42: /USB Audio Input/0V9BP -> 0V9
- U2 pad 49: /USB Audio Input/0V9BP -> 0V9
- U2 pad 52: /USB Audio Input/3V3BP -> +1V8
- U2 pad 57: /USB Audio Input/0V9BP -> 0V9
- U2 pad 61: /USB Audio Input/0V9BP -> 0V9
- U2 pad 62: /USB Audio Input/0V9BP -> 0V9
- U2 pad 63: /USB Audio Input/0V9BP -> 0V9
- U2 pad 64: /USB Audio Input/0V9BP -> 0V9
- U2 pad 8: /USB Audio Input/3V3BP -> +1V8
- U4 pad 1: Net-(U4A-+) -> /Headphone Amp Stage/OUTA
- U4 pad 2: Net-(U4A--) -> /DAC/DAC2b
- U4 pad 3: Net-(U4A-+) -> GND
- U4 pad 4: /Headphone Amp Stage/L-FLT -> /Audio Rails/+5V_FLT
- U4 pad 5: Net-(U4B-+) -> GND
- U4 pad 6: Net-(U4B--) -> /DAC/DAC2
- U4 pad 7: Net-(U4B-+) -> /Headphone Amp Stage/OUTB
- U5 pad 1: Net-(U5A-+) -> /Headphone Amp Stage/OUTC
- U5 pad 2: Net-(U5A--) -> /DAC/DAC1b
- U5 pad 3: Net-(U5A-+) -> GND
- U5 pad 4: /Headphone Amp Stage/L-FLT -> /Audio Rails/+5V_FLT
- U5 pad 5: Net-(U5B-+) -> GND
- U5 pad 6: Net-(U5B--) -> /DAC/DAC1
- U5 pad 7: Net-(U5B-+) -> /Headphone Amp Stage/OUTD
- U6 pad 1: /Low Noise Rails/Vin -> /Audio Rails/5Vin
- U6 pad 2: /Low Noise Rails/Vin -> /Audio Rails/5Vin
- U6 pad 3: /Low Noise Rails/Vin -> /Audio Rails/5Vin
- U7 pad 1: /Low Noise Rails/Vin -> /Audio Rails/5Vin
- U7 pad 2: /Low Noise Rails/Vin -> /Audio Rails/5Vin
- U7 pad 3: /Low Noise Rails/Vin -> /Audio Rails/5Vin
- U9 pad 4: /Low Noise Rails/Vin -> /Audio Rails/5Vin
Routing:
- net Net-(U4A-+): track 7.14 -> 0.00 mm, vias 2 -> 0
- net Net-(U5A-+): track 7.08 -> 0.00 mm, vias 2 -> 0
- net Net-(U4B-+): track 7.08 -> 0.00 mm, vias 2 -> 0
- net Net-(U5B-+): track 6.99 -> 0.00 mm, vias 2 -> 0
- net GND: track 0.00 -> 6.84 mm, vias 12 -> 8
- net Net-(U4B--): track 0.51 -> 0.00 mm

Commit message: Hopefully my mistakes are not for naught
Parts:
- moved Y2 109.2 mm to (36.0, 184.8)
- moved C3 108.0 mm to (55.0, 130.8)
- moved R15 107.1 mm to (32.5, 183.5)
- moved C24 104.8 mm to (36.0, 182.2), turned to 180 degrees
- moved C2 104.6 mm to (58.1, 126.3), turned to 90 degrees
- moved C95 102.8 mm to (56.1, 126.3), turned to 90 degrees
- moved R13 102.4 mm to (34.8, 173.2)
- moved C1 101.9 mm to (63.5, 127.5)
- moved C21 100.1 mm to (35.5, 168.8), turned to -90 degrees
- moved R17 99.7 mm to (39.5, 185.8)
- moved C20 96.9 mm to (42.5, 168.5), turned to -90 degrees
- moved C23 94.7 mm to (46.7, 175.5)
- moved R16 94.7 mm to (44.8, 180.8)
- moved J5 93.6 mm to (57.6, 140.1)
- moved Y3 92.8 mm to (47.0, 177.9)
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Connections:
- C45 pad 1: +1V8 -> Net-(U6-Sense)
- C61 pad 1: /Audio Rails/5Vin -> Net-(U6-Sense)
- U5 pad 5: GND -> unconnected-(U5B-+-Pad5)
- U5 pad 6: /DAC/DAC1 -> unconnected-(U5B---Pad6)
- U5 pad 7: /Headphone Amp Stage/OUTD -> unconnected-(U5-Pad7)
- U6 pad 7: +1V8 -> Net-(U6-Sense)
- U6 pad 8: +1V8 -> Net-(U6-Sense)
- U9 pad 1: unconnected-(U9-NC-Pad1) -> Net-(U6-Sense)
- U9 pad 3: unconnected-(U9-NC-Pad3) -> Net-(U6-Sense)
- U9 pad 4: /Audio Rails/5Vin -> unconnected-(U9-NC-Pad4)
Routing:
- net GND: track 6.84 -> 34.1 mm, vias 8 -> 24
- net /DAC/DAC_AVDD: track 0.00 -> 19.5 mm
- net +1.8V: track 0.00 -> 12.3 mm
- net /Clocking/XTAL1_OUT: track 0.00 -> 8.97 mm
- net /Debug/XMOS_NRST: track 0.00 -> 8.17 mm
- net +3.3V: track 0.00 -> 8.12 mm
- net Net-(U1-ADDR0): track 0.00 -> 6.89 mm
- net Net-(C20-Pad2): track 0.00 -> 6.48 mm
- net Net-(U6-Sense): track 0.00 -> 5.45 mm
- net Net-(U1-ADDR1): track 0.00 -> 3.61 mm
- net unconnected-(U5B-+-Pad5): track 0.00 -> 1.80 mm, vias 0 -> 1
