File: Headphone DAC AMP/_autosave-Headphone DAC AMP.kicad_pcb (KiCad board)
At the start: 4 copper layers, 55.2 x 67.7 mm, 63 parts, among them J3 SJ-3502-SMT, U1 ES9039Q2M, U2 TPS7A39, U3 TPA6120A2DWP, U4 OPA1612AxD, U5 OPA1612AxD, U6 TPS7A20xxxDQN

Commit message: Silk Changes
Parts:
- added G***: LOGO, LOGO, B.Cu at (87.5, 78.4)
- added G***: LOGO, LOGO, B.Cu at (127.5, 78.4)
- added G***: LOGO, LOGO, B.Cu at (87.5, 58.4)
- added G***: LOGO, LOGO, B.Cu at (87.5, 98.4)
- added G***: LOGO, LOGO, B.Cu at (107.5, 118.4)
- added G***: LOGO, LOGO, B.Cu at (87.5, 118.4)
- added G***: LOGO, LOGO, B.Cu at (107.5, 98.4)
- added G***: LOGO, LOGO, B.Cu at (127.5, 98.4)
- added G***: LOGO, LOGO, B.Cu at (107.5, 58.4)
- added G***: LOGO, LOGO, B.Cu at (107.5, 78.4)
- added G***: LOGO, LOGO, B.Cu at (127.5, 118.4)
- added G***: LOGO, LOGO, B.Cu at (127.5, 58.4)
